Commit message: Bringup robot complete

File: src/astrabot_description/urdf/bot_description.urdf.xacro (robot description, xacro)
@@ -15,4 +15,10 @@
   <xacro:property name="z_offset" value="-${base_height/2}" /> <!-- Space btw top of beam and the each joint -->
   <!-- Base Link -->
+  <link name="base_footprint"/>
+  <joint name="footprint_joint" type="fixed">
+    <parent link="base_footprint"/>
+    <child link="${prefix}base_link"/>
+    <origin xyz="0.0 0.0 0.05" rpy="0.0 0.0 0.0"/>
+  </joint>
   <link name="${prefix}base_link">
     <collision>

File: src/astrabot_description/urdf/bot_ros2_control.xacro (robot description, xacro)
@@ -3,9 +3,18 @@
   <xacro:macro name="diffbot_ros2_control" params="name prefix use_mock_hardware">
     <ros2_control name="${name}" type="system">
-      <!-- <xacro:unless value="${use_mock_hardware}">
+      <xacro:unless value="${use_mock_hardware}">
         <hardware>
-          <plugin>ros2_control_demo_example_2/DiffBotSystemHardware</plugin>
-          <param name="example_param_hw_start_duration_sec">0</param>
-          <param name="example_param_hw_stop_duration_sec">3.0</param>
+          <plugin>diffdrive_arduino/DiffDriveArduinoHardware</plugin>
+          <param name="left_wheel_name">left_wheel_joint</param>
+          <param name="right_wheel_name">right_wheel_joint</param>
+          <param name="loop_rate">30</param>
+          <param name="device">/dev/ttyUSB0</param>
+          <param name="baud_rate">57600</param>
+          <param name="timeout_ms">1000</param>
+          <param name="enc_counts_per_rev">2050</param>
+          <param name="pid_p">20</param>
+          <param name="pid_d">12</param>
+          <param name="pid_i">0</param>
+          <param name="pid_o">50</param>
         </hardware>
       </xacro:unless>
@@ -15,19 +24,5 @@
           <param name="calculate_dynamics">true</param>
         </hardware>
-      </xacro:if> -->
-      <hardware>
-        <plugin>diffdrive_arduino/DiffDriveArduinoHardware</plugin>
-        <param name="left_wheel_name">left_wheel_joint</param>
-        <param name="right_wheel_name">right_wheel_joint</param>
-        <param name="loop_rate">30</param>
-        <param name="device">/dev/serial/by-path/platform-fd500000.pcie-pci-0000:01:00.0-usb-0:1.3:1.0-port0</param>
-        <param name="baud_rate">57600</param>
-        <param name="timeout_ms">1000</param>
-        <param name="enc_counts_per_rev">3436</param>
-        <param name="pid_p">20</param>
-        <param name="pid_d">12</param>
-        <param name="pid_i">0</param>
-        <param name="pid_o">50</param>
-      </hardware>
+      </xacro:if>
       <joint name="${prefix}left_wheel_joint">
         <command_interface name="velocity"/>

Commit message: Complete

File: src/astrabot_description/urdf/bot_description.urdf.xacro (robot description, xacro)
@@ -44,4 +44,35 @@
       </inertial>
     </link>
+    <!-- LIDAR -->
+    <joint name="lidar_joint" type="fixed">
+      <parent link="${prefix}base_link"/>
+      <child link="${prefix}lidar_link"/>
+      <origin xyz="0.06 0.06 0.15" rpy="0.0 0.0 0.0"/>
+    </joint>
+    <link name="${prefix}lidar_link">
+      <visual>
+        <origin xyz="0 0 0" rpy="0 0 0"/>
+        <geometry>
+          <cylinder length="0.05" radius="0.025"/>
+        </geometry>
+        <material name="blue"/>
+      </visual>
+    </link>
+    <!-- IMU -->
+    <joint name="imu_joint" type="fixed">
+      <parent link="${prefix}base_link"/>
+      <child link="${prefix}imu_link"/>
+      <origin xyz="-0.04 -0.06 0.05" rpy="0.0 0.0 0.0"/>
+    </joint>
+    <link name="${prefix}imu_link">
+      <visual>
+        <origin xyz="0 0 0" rpy="0 0 0"/>
+        <geometry>
+          <cylinder length="0.01" radius="0.015"/>
+        </geometry>
+        <material name="blue"/>
+      </visual>
+    </link>
+    <!-- Wheels -->
     <joint name="${prefix}left_wheel_joint" type="continuous">
       <parent link="${prefix}base_link"/>
